File: implementation/checkpoint/interrupted.kicad_pcb (KiCad board)
At the start: 2 copper layers, 106 x 106 mm, 48 parts, among them IC1 74HCT14, IC2 74HCT74, IC3 UCC37321P, IC4 UCC37321P, IC6 78L05, J1 IEC C6, J110 Jumper 110V, J2 PE/CHASSIS, P1 PRIMARIO A, P2 PRIMARIO B, Q1 FGA60N65SMD, Q2 FGA60N65SMD, T1 1:1:1, T3 1:300

Commit message: fix(pcb): reroute HFBR and mains hole conflict with verified partial review
Routing:
- net +5V: track 75.7 -> 67.8 mm
- net /OPTICAL_OUT: track 21.9 -> 25.0 mm
Changed lines of the file:
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@@
 		)
 		(property "Value" "680u 35V"
-			(at 0 1.4 0)
+			(at 0 7.5 0)
 			(layer "F.Fab")
 			(effects
@@
 		)
 		(fp_text user "${REFERENCE}"
-			(at 0 -1.4 0)
+			(at 0 0 0)
 			(layer "F.Fab")
 			(effects
@@
 		)
 		(property "Value" "1000u 200V"
-			(at 0 1.4 0)
+			(at 0 16.25 0)
 			(layer "F.Fab")
 			(effects
@@
 		)
 		(fp_text user "${REFERENCE}"
-			(at 0 -1.4 0)
+			(at 0 0 0)
 			(layer "F.Fab")
 			(effects
@@
 		)
 		(property "Value" "100u 10V"
-			(at 0 1.4 180)
+			(at 0 5.25 180)
 			(layer "F.Fab")
 			(effects
@@
 		)
 		(fp_text user "${REFERENCE}"
-			(at 0 -1.4 180)
+			(at 0 0 180)
 			(layer "F.Fab")
 			(effects
@@
 		)
 		(property "Value" "100u 25V"
-			(at 0 1.4 0)
+			(at 0 5.25 0)
 			(layer "F.Fab")
 			(effects
@@
 		)
 		(fp_text user "${REFERENCE}"
-			(at 0 -1.4 0)
+			(at 0 0 0)
 			(layer "F.Fab")
 			(effects
@@
 		)
 		(property "Value" "100u 25V"
-			(at 0 1.4 0)
+			(at 0 5.25 0)
 			(layer "F.Fab")
 			(effects
@@
 		)
 		(fp_text user "${REFERENCE}"
-			(at 0 -1.4 0)
+			(at 0 0 0)
 			(layer "F.Fab")
 			(effects
@@
 		)
 		(property "Value" "1000u 200V"
-			(at 0 1.4 0)
+			(at 0 16.25 0)
 			(layer "F.Fab")
 			(effects
@@
 		)
 		(fp_text user "${REFERENCE}"
-			(at 0 -1.4 0)
+			(at 0 0 0)
 			(layer "F.Fab")
 			(effects
@@
 	)
 	(segment
-		(start 34 76)
-		(end 30 76)
+		(start 35.5 76)
+		(end 35.5 63.3)
 		(width 0.4064)
 		(layer "F.Cu")
@@
 	)
 	(segment
-		(start 30 63.5)
-		(end 27.305 63.5)
+		(start 34 76)
+		(end 35.5 76)
 		(width 0.4064)
 		(layer "F.Cu")
@@
 	)
 	(segment
-		(start 27.305 63.5)
-		(end 25.4 61.595)
+		(start 35.5 63.3)
+		(end 27.105 63.3)
 		(width 0.4064)
 		(layer "F.Cu")
@@
 	)
 	(segment
-		(start 30 76)
-		(end 30 63.5)
+		(start 27.105 63.3)
+		(end 25.4 61.595)
 		(width 0.4064)
 		(layer "F.Cu")
@@
 	)
 	(segment
-		(start 12 61.595)
-		(end 15.24 61.595)
-		(width 0.4064)
-		(layer "B.Cu")
-		(net "+5V")
-	)
-	(segment
 		(start 24.15 64.68)
 		(end 24.15 57)
@@
 	)
 	(segment
-		(start 12 57)
-		(end 12 61.595)
-		(width 0.4064)
-		(layer "B.Cu")
-		(net "+5V")
-	)
-	(segment
 		(start 34 68.38)
 		(end 32 68.38)
@@
 		(polygon
 			(pts
-				(xy 3.175 51.435) (xy 3.175 58) (xy 19.685 58) (xy 19.685 33.655) (xy 11.43 33.655) (xy 11.43 48.895)
+				(xy 3.175 51.435) (xy 3.175 66.675) (xy 19.685 66.675) (xy 19.685 33.655) (xy 11.43 33.655) (xy 11.43 48.895)
 				(xy 10.795 49.53) (xy 7.62 49.53) (xy 5.715 51.435)
 			)
