File: oneTesla.kicad_sch (KiCad schematic)
At the start: 42 parts, among them IC1 74HCT14, IC2 74HCT74, IC3 UCC37321P, IC4 UCC37321P, IC6 MC7805BDTRKG, J1 2EDGRC-5.08-02P, J110 Jumper 110V, J2 PE/CHASSIS, P1 PRIMARIO A, P2 PRIMARIO B, Q1 FGA60N65SMD, Q2 FGA60N65SMD, T1 1:1:1, T3 1:300

Commit message: Atualiza footprints dos capacitores e aterramento M3 do controle
Parts:
- C11, C12: footprint oneTesla:CP_D25_H45_P10.16_ReviewPending -> oneTesla:CP_SnapIn_D30.3_H40.5_P10.00_ReviewPending; Footprint_Status Ketuo 1000uF 200V, body D25 x H45mm from user image. Existi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 -> Snap-in: corpo D30.3 x H40.5mm; passo10mm e furos2mm confor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
- C9: value 100u 35V -> 10u 100V; footprint oneTesla:CP_Elec_8x10 -> oneTesla:C_1210_3225Metric; symbol oneTesla:C_Polarized -> oneTesla:C; Footprint_Status GENERIC: standard SMD 8x10mm selected as requested; purchas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 -> 10uF100V10%X7R1210 selected; standard3225 footprint; no man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
- J1: Assembly_Notes 1 = L; 2 = N. PE externo em J2/CHASSIS, separado de GND e D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 -> 1 = L; 2 = N. PE externo ao chassis e J2/GND CONTROLE; nunc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
- J2: value PE/CHASSIS -> PE / GND CONTROLE; footprint oneTesla:Chassis_PE_M3 -> oneTesla:PE_GND_Control_M3_D7.0mm; Assembly_Notes Entrada PE externa direta ao chassis por J2; J1 possui some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 -> PE da tomada ao ponto dedicado do chassis e ao terminal olh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; Footprint_Status REVIEW: Furo3.2 M3 pad5.1; cobre só0.2059 da borda; resistê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 -> Furo de fixacao da quina inferior esquerda reutilizado: (37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
Connections:
- net PE is gone; now on net GND: J2.1
Other:
- note added: "TERRA / PE: chassis metalico + J2 (GND CONTROLE). Nunca ligar a DC_MINUS, DC_MID ou SW_NODE."
Changed lines of the file:
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@@
 		)
 	)
-	(label "PE"
+	(label "GND"
 		(at 59.69 228.6 0)
 		(effects
@@
 	)
 	(symbol
-		(lib_id "oneTesla:C_Polarized")
+		(lib_id "oneTesla:C")
 		(at 201.93 222.25 0)
 		(unit 1)
@@
 			)
 		)
-		(property "Value" "100u 35V"
+		(property "Value" "10u 100V"
 			(at 205.74 222.6309 0)
 			(show_name no)
@@
 			)
 		)
-		(property "Footprint" "oneTesla:CP_Elec_8x10"
+		(property "Footprint" "oneTesla:C_1210_3225Metric"
 			(at 201.93 222.25 0)
 			(hide yes)
@@
 			)
 		)
-		(property "Description" ""
+		(property "Description" "MLCC10uF100V10%X7R1210, nonpolar; generic standard footprint"
 			(at 201.93 222.25 0)
+			(hide yes)
 			(show_name no)
 			(do_not_autoplace no)
@@
 			)
 		)
-		(property "Footprint_Status" "GENERIC: standard SMD 8x10mm selected as requested; purchased part dimensions unverified; pad1 positive, pad2 negative."
+		(property "Footprint_Status" "10uF100V10%X7R1210 selected; standard3225 footprint; no manufacturer-specific3D model."
 			(at 201.93 222.25 0)
 			(hide yes)
@@
 			)
 		)
-		(property "Assembly_Notes" "1 = L; 2 = N. PE externo em J2/CHASSIS, separado de GND e DC_MINUS."
+		(property "Assembly_Notes" "1 = L; 2 = N. PE externo ao chassis e J2/GND CONTROLE; nunca a DC_MINUS ou DC_MID."
 			(at 30.48 214.63 0)
 			(hide yes)
@@
 			)
 		)
-		(property "Footprint" "oneTesla:CP_D25_H45_P10.16_ReviewPending"
+		(property "Footprint" "oneTesla:CP_SnapIn_D30.3_H40.5_P10.00_ReviewPending"
 			(at 355.6 74.93 0)
 			(hide yes)
@@
 			)
 		)
-		(property "Footprint_Status" "Ketuo 1000uF 200V, body D25 x H45mm from user image. Existing P10.16mm, drill2mm and pad4mm preserved provisionally; actual terminal pitch and section NOT confirmed."
+		(property "Footprint_Status" "Snap-in: corpo D30.3 x H40.5mm; passo10mm e furos2mm conforme padrao recorrente Nichicon EL, Rubycon SN e Vishay PSM-SI; pads4mm."
 			(at 355.6 74.93 0)
 			(hide yes)
@@
 			)
 		)
-		(property "Value" "PE/CHASSIS"
+		(property "Value" "PE / GND CONTROLE"
 			(at 62.23 221.4879 0)
 			(show_name no)
@@
 			)
 		)
-		(property "Footprint" "oneTesla:Chassis_PE_M3"
+		(property "Footprint" "oneTesla:PE_GND_Control_M3_D7.0mm"
 			(at 59.69 223.52 0)
 			(hide yes)
@@
 			)
 		)
-		(property "Description" ""
+		(property "Description" "Entrada de terra de protecao ligada ao GND do controle, conforme topologia original oneTeslaTS."
 			(at 59.69 223.52 0)
+			(hide yes)
 			(show_name no)
 			(do_not_autoplace no)
@@
 			)
 		)
-		(property "Assembly_Notes" "Entrada PE externa direta ao chassis por J2; J1 possui somente L/N. Nao unir a GND ou DC_MINUS."
+		(property "Assembly_Notes" "PE da tomada ao ponto dedicado do chassis e ao terminal olhal no parafuso M3 de J2. J2 ligado ao GND do controle, nunca DC_MINUS/DC_MID. Contato metalico firme no cobre exposto; arruela/olhal ate D7mm, sem isolante entre contato e cobre; fixar cabo contra tracao."
 			(at 59.69 223.52 0)
 			(hide yes)
@@
 			)
 		)
-		(property "Footprint_Status" "REVIEW: Furo3.2 M3 pad5.1; cobre só0.2059 da borda; resistência/torque/arruela/bonding não definidos; F05"
+		(property "Footprint_Status" "Furo de fixacao da quina inferior esquerda reutilizado: (37.375,121.05)mm; PTH3.2mm, pad D7mm, olhal/arruela ate D7mm."
 			(at 59.69 223.52 0)
 			(hide yes)
@@
 			)
 		)
-		(property "Footprint" "oneTesla:CP_D25_H45_P10.16_ReviewPending"
+		(property "Footprint" "oneTesla:CP_SnapIn_D30.3_H40.5_P10.00_ReviewPending"
 			(at 355.6 120.65 0)
 			(hide yes)
@@
 			)
 		)
-		(property "Footprint_Status" "Ketuo 1000uF 200V, body D25 x H45mm from user image. Existing P10.16mm, drill2mm and pad4mm preserved provisionally; actual terminal pitch and section NOT confirmed."
+		(property "Footprint_Status" "Snap-in: corpo D30.3 x H40.5mm; passo10mm e furos2mm conforme padrao recorrente Nichicon EL, Rubycon SN e Vishay PSM-SI; pads4mm."
 			(at 355.6 120.65 0)
 			(hide yes)
@@
   )
 (label "SW_CT" (at 308.61 97.79 90) (effects (font (size 1.0 1.0)) (justify left bottom)))
+  (text "TERRA / PE: chassis metalico + J2 (GND CONTROLE).\nNunca ligar a DC_MINUS, DC_MID ou SW_NODE."
+    (at 18 235 0)
+    (effects (font (size 1.0 1.0)) (justify left top))
+)
 )

Commit message: Salva revisão DFM, arquivos de fabricação e modelos 3D completos
Parts:
- C12: footprint oneTesla:CP_SnapIn_D30.3_H40.5_P10.00_ReviewPending -> oneTesla:CP_SnapIn_D30.3_H40.5_P10.00_ReviewPending_DFM_C12
- C13: footprint oneTesla:CP_Elec_8x10 -> oneTesla:CP_Elec_8x10_DFM_C13
- C2: footprint oneTesla:C_0805_2012Metric_Pad1.18x1.45mm_HandSolder -> oneTesla:C_0805_2012Metric_Pad1.18x1.45mm_HandSolder_DFM_C2
- C8: footprint oneTesla:CP_Elec_8x10 -> oneTesla:CP_Elec_8x10_DFM_C8
- CPR1: footprint oneTesla:CDE_940C30S68K_F_CONFIRMAR -> oneTesla:CDE_940C30S68K_F_CONFIRMAR_DFM_CPR1
- D4: footprint oneTesla:Diode_Bridge_Vishay_KBU -> oneTesla:Diode_Bridge_Vishay_KBU_DFM_D4
- FB1: footprint oneTesla:HFBR-2521ETZ -> oneTesla:HFBR-2521ETZ_DFM_FB1
- IC3: footprint oneTesla:DIP-8_W7.62mm_Socket_LongPads -> oneTesla:DIP-8_W7.62mm_Socket_LongPads_DFM_IC3
- IC4: footprint oneTesla:DIP-8_W7.62mm_Socket_LongPads -> oneTesla:DIP-8_W7.62mm_Socket_LongPads_DFM_IC4
- J1: footprint oneTesla:TerminalBlock_2EDGRC-5.08_1x02_P5.08mm_Horizontal -> oneTesla:TerminalBlock_2EDGRC-5.08_1x02_P5.08mm_Horizontal_DFM_J1
- J110: footprint oneTesla:J110_WireLink_P15.24mm -> oneTesla:J110_WireLink_P15.24mm_DFM_J110
- J2: footprint oneTesla:PE_GND_Control_M3_D7.0mm -> oneTesla:PE_GND_Control_M3_D7.0mm_DFM_J2
- PS1: footprint oneTesla:HLK-15M15BL -> oneTesla:HLK-15M15BL_DFM_PS1
- Q1: footprint oneTesla:Q_TO3P_ImportedPads_ReviewPending -> oneTesla:Q_TO3P_ImportedPads_ReviewPending_DFM_Q1
- Q2: footprint oneTesla:Q_TO3P_ImportedPads_ReviewPending -> oneTesla:Q_TO3P_ImportedPads_ReviewPending_DFM_Q2
- R1: footprint oneTesla:R_Axial_Vishay_AC05_L18.0mm_D7.5mm_P10.16mm_Vertical -> oneTesla:R_Axial_Vishay_AC05_L18.0mm_D7.5mm_P10.16mm_Vertical_DFM_R1
- Z1: footprint oneTesla:D_DO201AD_P14.732_ReviewPending -> oneTesla:D_DO201AD_P14.732_ReviewPending_DFM_Z1
- Z2: footprint oneTesla:D_DO201AD_P14.732_ReviewPending -> oneTesla:D_DO201AD_P14.732_ReviewPending_DFM_Z2
Changed lines of the file:
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@@
 			)
 		)
-		(property "Footprint" "oneTesla:HFBR-2521ETZ"
+		(property "Footprint" "oneTesla:HFBR-2521ETZ_DFM_FB1"
 			(at 39.37 135.89 0)
 			(hide yes)
@@
 			)
 		)
-		(property "Footprint" "oneTesla:CP_Elec_8x10"
+		(property "Footprint" "oneTesla:CP_Elec_8x10_DFM_C13"
 			(at 168.91 168.91 0)
 			(hide yes)
@@
 			)
 		)
-		(property "Footprint" "oneTesla:Q_TO3P_ImportedPads_ReviewPending"
+		(property "Footprint" "oneTesla:Q_TO3P_ImportedPads_ReviewPending_DFM_Q1"
 			(at 294.64 74.93 0)
 			(hide yes)
@@
 			)
 		)
-		(property "Footprint" "oneTesla:HLK-15M15BL"
+		(property "Footprint" "oneTesla:HLK-15M15BL_DFM_PS1"
 			(at 118.11 217.17 0)
 			(hide yes)
@@
 			)
 		)
-		(property "Footprint" "oneTesla:C_0805_2012Metric_Pad1.18x1.45mm_HandSolder"
+		(property "Footprint" "oneTesla:C_0805_2012Metric_Pad1.18x1.45mm_HandSolder_DFM_C2"
 			(at 344.17 218.44 0)
 			(hide yes)
@@
 			)
 		)
-		(property "Footprint" "oneTesla:TerminalBlock_2EDGRC-5.08_1x02_P5.08mm_Horizontal"
+		(property "Footprint" "oneTesla:TerminalBlock_2EDGRC-5.08_1x02_P5.08mm_Horizontal_DFM_J1"
 			(at 30.48 214.63 0)
 			(hide yes)
@@
 			)
 		)
-		(property "Footprint" "oneTesla:CP_Elec_8x10"
+		(property "Footprint" "oneTesla:CP_Elec_8x10_DFM_C8"
 			(at 133.35 168.91 0)
 			(hide yes)
@@
 			)
 		)
-		(property "Footprint" "oneTesla:CP_SnapIn_D30.3_H40.5_P10.00_ReviewPending"
+		(property "Footprint" "oneTesla:CP_SnapIn_D30.3_H40.5_P10.00_ReviewPending_DFM_C12"
 			(at 355.6 74.93 0)
 			(hide yes)
@@
 			)
 		)
-		(property "Footprint" "oneTesla:Diode_Bridge_Vishay_KBU"
+		(property "Footprint" "oneTesla:Diode_Bridge_Vishay_KBU_DFM_D4"
 			(at 46.99 262.89 90)
 			(hide yes)
@@
 			)
 		)
-		(property "Footprint" "oneTesla:DIP-8_W7.62mm_Socket_LongPads"
+		(property "Footprint" "oneTesla:DIP-8_W7.62mm_Socket_LongPads_DFM_IC4"
 			(at 196.85 137.16 0)
 			(hide yes)
@@
 			)
 		)
-		(property "Footprint" "oneTesla:D_DO201AD_P14.732_ReviewPending"
+		(property "Footprint" "oneTesla:D_DO201AD_P14.732_ReviewPending_DFM_Z1"
 			(at 322.58 74.93 90)
 			(hide yes)
@@
 			)
 		)
-		(property "Footprint" "oneTesla:DIP-8_W7.62mm_Socket_LongPads"
+		(property "Footprint" "oneTesla:DIP-8_W7.62mm_Socket_LongPads_DFM_IC3"
 			(at 196.85 58.42 0)
 			(hide yes)
@@
 			)
 		)
-		(property "Footprint" "oneTesla:PE_GND_Control_M3_D7.0mm"
+		(property "Footprint" "oneTesla:PE_GND_Control_M3_D7.0mm_DFM_J2"
 			(at 59.69 223.52 0)
 			(hide yes)
@@
 			)
 		)
-		(property "Footprint" "oneTesla:J110_WireLink_P15.24mm"
+		(property "Footprint" "oneTesla:J110_WireLink_P15.24mm_DFM_J110"
 			(at 106.68 264.16 0)
 			(hide yes)
@@
 			)
 		)
-		(property "Footprint" "oneTesla:Q_TO3P_ImportedPads_ReviewPending"
+		(property "Footprint" "oneTesla:Q_TO3P_ImportedPads_ReviewPending_DFM_Q2"
 			(at 294.64 120.65 0)
 			(hide yes)
@@
 			)
 		)
-		(property "Footprint" "oneTesla:R_Axial_Vishay_AC05_L18.0mm_D7.5mm_P10.16mm_Vertical"
+		(property "Footprint" "oneTesla:R_Axial_Vishay_AC05_L18.0mm_D7.5mm_P10.16mm_Vertical_DFM_R1"
 			(at 46.99 73.66 90)
 			(hide yes)
@@
 			)
 		)
-		(property "Footprint" "oneTesla:CDE_940C30S68K_F_CONFIRMAR"
+		(property "Footprint" "oneTesla:CDE_940C30S68K_F_CONFIRMAR_DFM_CPR1"
 			(at 312.42 97.79 90)
 			(hide yes)
@@
 			)
 		)
-		(property "Footprint" "oneTesla:D_DO201AD_P14.732_ReviewPending"
+		(property "Footprint" "oneTesla:D_DO201AD_P14.732_ReviewPending_DFM_Z2"
 			(at 322.58 120.65 90)
 			(hide yes)
